Commit message: gmapping

File: src/fourbot/urdf/temp_fourbot.xacro (robot description, xacro)
@@ -10,7 +10,7 @@
 	<xacro:property name="robot_wheel_length" value="0.05"/>
 	<xacro:property name="robot_wheel_radius" value="0.1"/>
-	<!-- <xacro:property name="camera_mass" value="0.1"/> -->
+	<xacro:property name="camera_mass" value="0.1"/>
 	<xacro:property name="hokoyu_mass" value="1e-5"/>
-	<!-- <xacro:property name="depthcam_mass" value="1e-5"/> -->
+	<xacro:property name="depthcam_mass" value="1e-5"/>
 	<!-- Make Chassis of Bot -->
 	<link name="chassis">
@@ -159,5 +159,5 @@
 	</link> -->
 	<!-- Hokuyo Lidar -->
-	<link name="hokuyo">
+	<!-- <link name="hokuyo">
 		<inertial>
 			<mass value="${hokoyu_mass}"/>
@@ -181,5 +181,5 @@
 			</geometry>
 		</collision>
-	</link>
+	</link> -->
 	<!-- Depth Cam Kinect Link -->
 	<!-- <link name="depthcam">
@@ -253,10 +253,10 @@
 	</joint> -->
 	<!-- Hokoyu Joint -->
-	<joint name="hokuyo_joint" type="fixed">
+	<!-- <joint name="hokuyo_joint" type="fixed">
 	    <origin xyz="0.2 0 0.2" rpy="0 0 0" />
 	    <parent link="chassis"/>
 	    <child link="hokuyo" />
 	    <axis xyz="0 1 0"/>
-	</joint>
+	</joint> -->
 	<!-- Depth Sensor Cam Joint -->
 	<!-- <joint name="depthcam_joint" type="fixed">
@@ -315,7 +315,98 @@
 		<material>Gazebo/Black</material>
 	</gazebo> -->
+	<gazebo reference="ouster_lidar">
+		<material>Gazebo/Black</material>
+	</gazebo>
 	<gazebo reference="chassis">
 		<material>Gazebo/Blue</material>
 	</gazebo>
-	<xacro:include filename="$(find fourbot)/urdf/fourbot.gazebo" />
+	<gazebo reference="ouster_lidar">
+		<sensor type="ray" name="ouster_lidar">
+		  <pose>0 0 0 0 0 0</pose>
+		  <visualize>false</visualize>
+		  <update_rate>10</update_rate>
+		  <ray>
+			<scan>
+			  <vertical>
+			  <samples>64</samples>
+			  <resolution>1</resolution>
+			  <min_angle>${-16.6*3.1415926535897931/180.0}</min_angle>
+			  <max_angle>${16.6*3.1415926535897931/180.0}</max_angle>
+			  </vertical>
+			  <horizontal>
+			  <samples>512</samples>
+			  <resolution>1</resolution>
+			  <min_angle>-3.1415926535897931</min_angle>
+			  <max_angle>3.1415926535897931</max_angle>
+			  </horizontal>
+			</scan>
+			<range>
+				<min>0.8</min>
+				<max>100</max>
+				<resolution>0.03</resolution>
+			</range>
+			<noise>
+			  <type>gaussian</type>
+			  <mean>0.0</mean>
+			  <stddev>0.000000000001</stddev>
+			</noise>
+		  </ray>
+		  <plugin name="gazebo_ros_laser_controller" filename="libgazebo_ros_ouster_laser.so">
+			<topicName>fourbot/os1_cloud_node/points</topicName>
+			<frameName>ouster_lidar</frameName>
+			<min_range>0.8</min_range>
+			<max_range>100</max_range>
+			<gaussianNoise>0.008</gaussianNoise>
+		  </plugin>
+		</sensor>
+		</gazebo>
+		<gazebo reference="ouster_imu">
+			<sensor type="imu" name="ouster_imu_sensor">
+			  <pose>0 0 0 0 0 0</pose>
+			  <always_on>true</always_on>
+			  <update_rate>100</update_rate>
+			  <visualize>true</visualize>
+			  <topic>fourbot/os1_cloud_node/imu</topic>
+			</sensor>
+		</gazebo>
+		<!-- Ouster 3D Lidar -->
+		<xacro:property name="file_visual" value="os1_64_reduced"/>
+		<xacro:property name="gpu_str" value=""/>
+		<joint name="ouster_joint" type="fixed">
+			<origin xyz="0 0 0" rpy="0 0 0" />
+			<parent link="chassis"/>
+			<child link="ouster_sensor"/>
+		</joint>
+		<link name="ouster_sensor">
+			<inertial>
+				<mass value="0.425"/>
+				<origin xyz="0 0 0.13675" rpy="0 0 0" />
+				<inertia ixx="0.000308429" ixy="0" ixz="0"
+						iyy="0.000308429" iyz="0" izz="0.00034589"/>
+			</inertial>
+			<collision name="lidar_collision">
+				<origin xyz="0 0 0.13675" rpy="0 0 0" />
+				<geometry>
+				<cylinder radius="0.04350" length="0.07350"/>
+				</geometry>
+			</collision>
+			<visual name="lidar_visual">
+				<origin xyz="0 0 0.13675" rpy="0 0 0"/>
+				<geometry>
+				<mesh filename="package://fourbot/meshes/${file_visual}.stl" />
+				</geometry>
+			</visual>
+		</link>
+		<link name="ouster_lidar">
+			<pose>0 0 0 0 0 3.1415926535897931</pose>
+		</link>
+		<joint name="ouster_lidar_joint" type="fixed">
+			<parent link="ouster_sensor"/>
+			<child link="ouster_lidar"/>
+		</joint>
+		<link name="ouster_imu"/>
+		<joint name="ouster_imu_joint" type="fixed">
+			<parent link="ouster_sensor"/>
+			<child link="ouster_imu"/>
+		</joint>
 </robot>
